Commit message: chore: fred complete description

File: src/description/fred_description.urdf (robot description, URDF)
Before this commit: robot frederico, 3 links, 2 joints
Links:
- removed link base_footprint
- removed link front_caster
- added link lidar_link
- added link roda1_link, mass 0.429989283650456; collision mesh filename=file:///home/ubuntu/ros2_ws/src/fred2_description/meshes/ro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; visual mesh filename=file:///home/ubuntu/ros2_ws/src/fred2_description/meshes/ro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
- added link roda2, mass 0.429989283650456; collision mesh filename=file:///home/ubuntu/ros2_ws/src/fred2_description/meshes/ro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; visual mesh filename=file:///home/ubuntu/ros2_ws/src/fred2_description/meshes/ro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
- added link roda3, mass 0.429989283650456; collision mesh filename=file:///home/ubuntu/ros2_ws/src/fred2_description/meshes/ro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; visual mesh filename=file:///home/ubuntu/ros2_ws/src/fred2_description/meshes/ro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
- added link roda4, mass 0.429989283650456; collision mesh filename=/home/ubuntu/ros2_ws/src/fred2_description/meshes/roda4.STL; visual mesh filename=file:///home/ubuntu/ros2_ws/src/fred2_description/meshes/ro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
- link base_link: mass None -> 4.63143329848068; geometry collision mesh filename=file:///home/ubuntu/ros2_ws/src/fred2_description/meshes/ba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; visual mesh filename=file:///home/ubuntu/ros2_ws/src/fred2_description/meshes/ba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
Joints:
- removed joint base_joint
- removed joint caster_joint
- added joint lidar_joint: type fixed, parent base_link, child lidar_link, origin xyz=0 0.18 0.187 rpy=0 0 0
- added joint roda1: type continuous, parent base_link, child roda1_link, origin xyz=0.14881 0.113 0.025 rpy=1.5708 -1.3493 1.5708, axis 0 0 1
- added joint roda2: type continuous, parent base_link, child roda2, origin xyz=-0.14881 0.113 0.025 rpy=1.5708 1.3493 -1.5708, axis 0 0 1
- added joint roda3: type continuous, parent base_link, child roda3, origin xyz=0.14881 -0.113 0.025 rpy=1.5708 0.72582 1.5708, axis 0 0 1
- added joint roda4: type continuous, parent base_link, child roda4, origin xyz=-0.14881 -0.113 0.025 rpy=1.5708 -0.72582 -1.5708, axis 0 0 1
